Commit message: URDF skeleton for 6-DOF arm

File: src/pandalite_description/urdf/pandalite.urdf (robot description, URDF)
Before this commit: robot pandalite, 2 links, 1 joints
Links:
- added link link_2, mass 0.4; visual cylinder length=0.18 radius=0.025
- added link link_3, mass 0.3; visual cylinder length=0.18 radius=0.022
- added link link_4, mass 0.15; visual box size=0.04 0.05 0.03
- added link link_5, mass 0.12; visual box size=0.04 0.03 0.05
- added link link_6, mass 0.1; visual box size=0.04 0.05 0.03
- added link tool_tip, mass 0.001
Joints:
- added joint link_1_2_joint: type revolute, parent link_1, child link_2, origin xyz=0 0 0.06 rpy=0 0 0, axis 0 1 0, limit lower=-2.0 upper=2.0 effort=10.0 velocity=2.5
- added joint link_2_3_joint: type revolute, parent link_2, child link_3, origin xyz=0.18 0 0 rpy=0 0 0, axis 0 1 0, limit lower=-2.5 upper=2.5 effort=8.0 velocity=2.5
- added joint link_3_4_joint: type revolute, parent link_3, child link_4, origin xyz=0.18 0 0 rpy=0 0 0, axis 1 0 0, limit lower=-3.14 upper=3.14 effort=5.0 velocity=3.0
- added joint link_4_5_joint: type revolute, parent link_4, child link_5, origin xyz=0.04 0 0 rpy=0 0 0, axis 0 1 0, limit lower=-2.0 upper=2.0 effort=4 velocity=3
- added joint tool_tip_joint: type fixed, parent link_6, child tool_tip, origin xyz=0.04 0 0 rpy=0 0 0
- added joint wrist_yaw: type revolute, parent link_5, child link_6, origin xyz=0.04 0 0 rpy=0 0 0, axis 0 0 1, limit lower=-3.14 upper=3.14 effort=3.0 velocity=3.0
